File: uSlime_PCB/power.kicad_sch (KiCad schematic)
At the start: 20 parts, among them CN2 1.25T-2AW, J1 USB_C_Receptacle_USB2.0_14P, U2 MSK-12C02_SMD_SPDT_SWITCH, U3 AP2112K-3.3TRG1, U4 MCP73831T-2ACI/OT

Commit message: v0.0.2a Modify BNO I2C
Parts:
- D1, D2: footprint Diode_SMD:D_0402_1005Metric -> uSlime-libs:D_0402_1005Metric
Changed lines of the file:
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@@
 			)
 		)
-		(property "Footprint" "Diode_SMD:D_0402_1005Metric"
+		(property "Footprint" "uSlime-libs:D_0402_1005Metric"
 			(at 67.31 71.12 0)
 			(effects
@@
 			)
 		)
-		(property "Footprint" "Diode_SMD:D_0402_1005Metric"
+		(property "Footprint" "uSlime-libs:D_0402_1005Metric"
 			(at 57.15 77.47 0)
 			(effects
