File: uSlime_PCB_Module/BNO085.kicad_sch (KiCad schematic)
At the start: 9 parts, among them CN1 X1502WR-05K-N0SN, U5 BNO085

Commit message: Add module version
Parts:
- removed C6, C9: 0.1uF, Capacitor_SMD:C_0402_1005Metric, symbol uSlime:C
- removed JP1: Jumper_3_Open, Jumper:SolderJumper-3_P1.3mm_Open_RoundedPad1.0x1.5mm, symbol uSlime:Jumper_3_Open
- removed R10, R9: 2.2k, Resistor_SMD:R_0402_1005Metric, symbol uSlime:R_US
- removed R11, R12: 10k, Resistor_SMD:R_0402_1005Metric, symbol uSlime:R_US
- removed U5: BNO085, uSlime-libs:BNO080, symbol uSlime:BNO085
- added J2: Conn_01x05, Connector_PinHeader_2.54mm:PinHeader_1x05_P2.54mm_Vertical, symbol uSlime:Conn_01x05
Connections:
- net +3.3V: now also J2.4 (Pin_4)
- net BNO_INT: now also J2.3 (Pin_3)
- net BNO_SCL: now also J2.1 (Pin_1)
- net BNO_SDA: now also J2.5 (Pin_5)
- net GND: now also J2.2 (Pin_2)
- no-connect marks 4 -> 0
