File: uSlime_PCB_Module/uSlime_PCB_Module.kicad_pcb (KiCad board)
At the start: 2 copper layers, 25 x 35.6 mm, 57 parts, among them CN1 X1502WR-05K-N0SN, CN2 1.25T-2AW, J1 USB_C_Receptacle_USB2.0_14P, U1 BNO085, U1 ESP32-C6-MINI-1, U2 MSK-12C02_SMD_SPDT_SWITCH, U3 AP2112K-3.3TRG1, U4 MCP73831T-2ACI/OT, U5 BNO085

Commit message: Add module version
Parts:
- removed the C1 at (107.8, 119.2)
- removed the C2 at (107.8, 118.3)
- removed the C3 at (110.0, 119.7)
- removed the C4 at (112.4, 123.9)
- removed C6, C9: 0.1uF, Capacitor_SMD:C_0402_1005Metric
- removed the CN1 at (113.5, 117.2)
- removed the G*** at (111.6, 121.2)
- removed JP1 (x2): Jumper_3_Open, Jumper:SolderJumper-3_P1.3mm_Open_RoundedPad1.0x1.5mm
- removed the R1 at (110.0, 121.5)
- removed R10, R9: 2.2k, Resistor_SMD:R_0402_1005Metric
- removed R11, R12: 10k, Resistor_SMD:R_0402_1005Metric
- removed the R2 at (114.3, 123.9)
- removed the R3 at (107.7, 117.3)
- removed the R4 at (117.5, 119.3)
- removed REF** (x2): NPTH, PCM_kikit:NPTH
- removed the U1 at (113.5, 121.0)
- removed U5: BNO085, uSlime-libs:BNO080
- added J2: Conn_01x05, Connector_PinHeader_2.54mm:PinHeader_1x05_P2.54mm_Vertical, B.Cu at (123.3, 104.0)
- moved RESET1 8.41 mm to (114.4, 107.5), turned to 90 degrees
- moved R2 6.40 mm to (113.0, 101.7), turned to 180 degrees
- moved C1 4.12 mm to (114.9, 101.7), turned to 0 degrees
- moved R7 2.28 mm to (112.2, 108.6)
- moved C2 0.32 mm to (120.3, 101.5)
- moved STAT1 0.32 mm to (122.2, 101.5)
- moved R8 0.32 mm to (124.1, 101.5)
- moved R6 0.11 mm to (112.2, 106.7), turned to 90 degrees
Routing:
- net +3.3V: track 99.9 -> 50.2 mm, vias 6 -> 3
- net GND: track 139.0 -> 103.0 mm, vias 8 -> 4
- net Net-(JP1-C): track 23.7 -> 0.00 mm, vias 3 -> 0
- net BNO_SCL: track 44.6 -> 26.6 mm
- net BNO_SDA: track 45.3 -> 29.1 mm, vias 5 -> 2
- net BNO_INT2: track 32.1 -> 18.7 mm, vias 2 -> 1
- net Net-(U5-BOOTN): track 8.91 -> 0.00 mm, vias 2 -> 0
- net Net-(U5-NRST): track 8.18 -> 0.00 mm, vias 2 -> 0
- net /ESP32-C6FH4/ESP_EN: track 16.0 -> 20.9 mm, vias 2 -> 3
- net (no net): track 4.29 -> 0.00 mm
- net BNO_INT: track 10.4 -> 7.69 mm
- net Net-(U5-CAP): track 2.47 -> 0.00 mm
- net Net-(J1-CC2): track 9.90 -> 8.80 mm
- net Net-(J1-CC1): track 10.7 -> 9.64 mm
Other:
- board size 25 x 35.6 mm -> 25 x 22.6 mm
- board text removed: "0x4A"
- board text removed: "0x4B"
- board text removed: "Slime"
